File: Netzteil.kicad_pcb (KiCad board)
At the start: 2 copper layers, 61 x 27 mm, 15 parts, among them J1 Conn_01x02_Socket, J2 Conn_01x02_Socket, J3 J-jumper, P1 P-trim, U1 LM2596S-ADJ

Commit message: First Routes.
Parts:
- moved C4 6.80 mm to (171.5, 59.0)
- moved D3 3.33 mm to (147.9, 69.2), turned to 180 degrees
- moved C3 2.83 mm to (167.5, 60.3)
- moved R1 2.69 mm to (142.0, 69.5), turned to 180 degrees
- moved C2 2.00 mm to (137.5, 64.7)
- turned C1 to -90 degrees
- turned D2 to 180 degrees
Routing:
- net Net-(C3-+): track 0.00 -> 52.7 mm
- net Net-(C1-+): track 0.00 -> 19.9 mm
- net Net-(P1-a): track 0.00 -> 19.4 mm
- net +VDC: track 0.00 -> 17.3 mm
- net Net-(D3-A): track 0.00 -> 9.47 mm
- net Net-(C2-+): track 0.00 -> 6.21 mm
- net Net-(U1-~{ON}/OFF): track 0.00 -> 5.92 mm
- added copper zone on F.Cu, net V-GND
Other:
- board size 61 x 27 mm -> 61 x 27.5 mm

Commit message: Second try routing.
Parts:
- added REF**: MountingHole_3.5mm, MountingHole:MountingHole_3.5mm, F.Cu at (165.0, 51.0)
- added REF**: MountingHole_3.5mm, MountingHole:MountingHole_3.5mm, F.Cu at (120.5, 69.5)
- added REF**: MountingHole_3.5mm, MountingHole:MountingHole_3.5mm, F.Cu at (120.5, 51.5)
- added REF**: MountingHole_3.5mm, MountingHole:MountingHole_3.5mm, F.Cu at (165.0, 69.5)
- moved D3 20.3 mm to (127.8, 66.9), turned to -90 degrees
- moved J3 15.3 mm to (140.5, 67.5), turned to 90 degrees
- moved C4 12.7 mm to (159.0, 61.5)
- moved C3 12.1 mm to (155.5, 61.5)
- moved D4 10.1 mm to (152.0, 64.5)
- moved R1 9.85 mm to (133.0, 65.5)
- moved C2 8.29 mm to (130.5, 60.3)
- moved J1 7.07 mm to (120.5, 59.0), turned to -90 degrees
- moved P1 5.85 mm to (155.5, 55.6)
- moved J2 5.21 mm to (165.0, 62.5), turned to 90 degrees
- moved D1 5.15 mm to (127.5, 60.5)
- moved C1 4.42 mm to (134.5, 60.5)
- moved L1 3.91 mm to (130.0, 52.5)
- moved U1 3.85 mm to (143.7, 54.4)
- moved D2 2.92 mm to (126.0, 52.5), turned to -90 degrees
Routing:
- net Net-(U1-~{ON}/OFF): track 5.92 -> 16.7 mm
- net Net-(C2-+): track 6.21 -> 12.0 mm
- net Net-(P1-a): track 19.4 -> 14.1 mm
- net Net-(D3-A): track 9.47 -> 4.91 mm
- net +VDC: track 17.3 -> 13.9 mm
- net Net-(C1-+): track 19.9 -> 17.3 mm
- net Net-(C3-+): track 52.7 -> 53.8 mm
Other:
- board size 61 x 27.5 mm -> 52.5 x 26 mm

Commit message: PCB design correction
Parts:
- moved J1 1.00 mm to (121.5, 59.0)
- moved J2 0.71 mm to (164.5, 63.0)
- moved P1 0.50 mm to (155.5, 56.1)
Routing:
- net Net-(P1-a): track 14.1 -> 17.5 mm
- net +VDC: track 13.9 -> 11.9 mm
- net Net-(D3-A): track 4.91 -> 4.16 mm
Other:
- board text added: "RasPower 0.2 © Kroesch.NET"
- board text added: "Vin + 9~24V"
- board text added: "Vout +"
Changed lines of the file:
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@@
 	(footprint "TerminalBlock_Phoenix:TerminalBlock_Phoenix_MPT-0,5-2-2.54_1x02_P2.54mm_Horizontal"
 		(layer "F.Cu")
-		(at 165 62.54 90)
+		(at 164.46 63 90)
 		(descr "Terminal Block Phoenix MPT-0,5-2-2.54, 2 pins, pitch 2.54mm, size 5.54x6.2mm, drill diameter 1.1mm, pad diameter 2.2mm, http://www.mouser.com/ds/2/324/ItemDetail_1725656-920552.pdf, script-generated using https://gitlab.com/kicad/libraries/kicad-footprint-generator/-/tree/master/scripts/TerminalBlock_Phoenix")
 		(tags "THT Terminal Block Phoenix MPT-0,5-2-2.54 pitch 2.54mm size 5.54x6.2mm drill 1.1mm pad 2.2mm")
@@
 			(at 1.27 -4.22 90)
 			(layer "F.SilkS")
+			(hide yes)
 			(effects
 				(font
@@
 			(at 1.27 4.22 90)
 			(layer "F.Fab")
+			(hide yes)
 			(effects
 				(font
@@
 		(tags "Inductor Radial series Radial pin pitch 5.00mm  diameter 7.5mm height 12.5mm Fastron 07P")
 		(property "Reference" "L1"
-			(at 2.5 -5 0)
+			(at 2.5 -2.5 0)
 			(layer "F.SilkS")
 			(effects
@@
 		(tags "capacitor tantalum")
 		(property "Reference" "C4"
-			(at 0 -2.35 90)
+			(at 3.46 0 180)
 			(layer "F.SilkS")
 			(effects
@@
 	(footprint "Potentiometer_THT:Potentiometer_Bourns_3386P_Vertical"
 		(layer "F.Cu")
-		(at 155.5 55.58)
+		(at 155.5 56.08)
 		(descr "Potentiometer, vertical, Bourns 3386P, https://www.bourns.com/pdfs/3386.pdf")
 		(tags "Potentiometer vertical Bourns 3386P")
 		(property "Reference" "P1"
-			(at -0.015 -8.555 0)
+			(at 3.5 -6.08 0)
 			(layer "F.SilkS")
 			(effects
@@
 			(at 0 -4.5 0)
 			(layer "F.SilkS")
+			(hide yes)
 			(effects
 				(font
@@
 		(tags "capacitor")
 		(property "Reference" "C3"
-			(at 0 -1.43 90)
+			(at 2.5 -0.5 180)
 			(layer "F.SilkS")
 			(effects
@@
 		(tags "Diode SMA (DO-214AC)")
 		(property "Reference" "D1"
-			(at 0 -2.5 90)
+			(at 2.5 -2.49 90)
 			(layer "F.SilkS")
 			(effects
@@
 		(tags "Diode SMA (DO-214AC)")
 		(property "Reference" "D4"
-			(at 0 -2.5 90)
+			(at 2.5 -3 180)
 			(layer "F.SilkS")
 			(effects
@@
 		(tags "dual led smd")
 		(property "Reference" "D3"
-			(at 0 -2.5 90)
+			(at -0.9 2.275 90)
 			(layer "F.SilkS")
 			(effects
@@
 		(tags "Diode SMA (DO-214AC)")
 		(property "Reference" "D2"
-			(at 0 -2.5 90)
+			(at 3 2 90)
 			(layer "F.SilkS")
 			(effects
@@
 	(footprint "TerminalBlock_Phoenix:TerminalBlock_Phoenix_MPT-0,5-2-2.54_1x02_P2.54mm_Horizontal"
 		(layer "F.Cu")
-		(at 120.5 59 -90)
+		(at 121.5 58.96 -90)
 		(descr "Terminal Block Phoenix MPT-0,5-2-2.54, 2 pins, pitch 2.54mm, size 5.54x6.2mm, drill diameter 1.1mm, pad diameter 2.2mm, http://www.mouser.com/ds/2/324/ItemDetail_1725656-920552.pdf, script-generated using https://gitlab.com/kicad/libraries/kicad-footprint-generator/-/tree/master/scripts/TerminalBlock_Phoenix")
 		(tags "THT Terminal Block Phoenix MPT-0,5-2-2.54 pitch 2.54mm size 5.54x6.2mm drill 1.1mm pad 2.2mm")
 		(property "Reference" "J1"
-			(at 1.27 -4.22 90)
+			(at -2.46 0 180)
 			(layer "F.SilkS")
 			(effects
@@
 		(layer "Edge.Cuts")
 	)
+	(gr_text "RasPower 0.2\n© Kroesch.NET"
+		(at 150 72.5 0)
+		(layer "F.SilkS")
+		(effects
+			(font
+				(size 1 1)
+				(thickness 0.1)
+			)
+			(justify left bottom)
+		)
+	)
+	(gr_text "Vin +\n9~24V"
+		(at 118 66.5 0)
+		(layer "F.SilkS")
+		(effects
+			(font
+				(size 1 1)
+				(thickness 0.1)
+			)
+			(justify left bottom)
+		)
+	)
+	(gr_text "Vout +"
+		(at 162.5 66.5 0)
+		(layer "F.SilkS")
+		(effects
+			(font
+				(size 1 1)
+				(thickness 0.1)
+			)
+			(justify left bottom)
+		)
+	)
 	(segment
 		(start 135 52.5)
@@
 	)
 	(segment
+		(start 162.46 60)
+		(end 162.46 61)
+		(width 0.2)
+		(layer "F.Cu")
+		(net 4)
+	)
+	(segment
 		(start 152 62.5)
 		(end 153.725 62.5)
@@
 	)
 	(segment
-		(start 162.46 60)
-		(end 165 62.54)
+		(start 162.46 61)
+		(end 164.46 63)
 		(width 0.2)
 		(layer "F.Cu")
@@
 	)
 	(segment
-		(start 126 57)
-		(end 127.5 58.5)
+		(start 127.5 58.5)
+		(end 126 57)
 		(width 0.2)
 		(layer "F.Cu")
@@
 	)
 	(segment
-		(start 126 56.04)
-		(end 126 54.5)
+		(start 126.5 58.5)
+		(end 127.5 58.5)
 		(width 0.2)
 		(layer "F.Cu")
@@
 	)
 	(segment
-		(start 120.5 61.54)
-		(end 126 56.04)
+		(start 126 57)
+		(end 126 54.5)
 		(width 0.2)
 		(layer "F.Cu")
@@
 	)
 	(segment
-		(start 126 54.5)
-		(end 126 57)
+		(start 121.5 61.5)
+		(end 123.5 61.5)
 		(width 0.2)
 		(layer "F.Cu")
@@
 	)
 	(segment
-		(start 128.7 68.3)
-		(end 128.5 68.3)
+		(start 123.5 61.5)
+		(end 126.5 58.5)
 		(width 0.2)
 		(layer "F.Cu")
-		(net 6)
+		(net 5)
 	)
 	(segment
-		(start 133.5 65.5)
-		(end 133.5 66.25)
+		(start 128.7 68.3)
+		(end 128.5 68.3)
 		(width 0.2)
 		(layer "F.Cu")
@@
 	)
 	(segment
-		(start 145.425 62.075)
-		(end 145.425 59.775)
+		(start 145.425 59.775)
+		(end 147.274 57.926)
 		(width 0.2)
 		(layer "F.Cu")
@@
 	)
 	(segment
-		(start 153.154 57.926)
-		(end 155.5 55.58)
+		(start 153.654 57.926)
+		(end 155.5 56.08)
+		(width 0.2)
+		(layer "F.Cu")
+		(net 8)
+	)
+	(segment
+		(start 145.425 62.075)
+		(end 145.425 59.775)
 		(width 0.2)
 		(layer "F.Cu")
@@
 	(segment
 		(start 147.274 57.926)
-		(end 153.154 57.926)
+		(end 153.654 57.926)
 		(width 0.2)
 		(layer "F.Cu")
@@
 	)
 	(segment
-		(start 145.425 59.775)
-		(end 147.274 57.926)
+		(start 158.04 53.54)
+		(end 155.5 56.08)
 		(width 0.2)
 		(layer "F.Cu")
