File: Netzteil.kicad_sch (KiCad schematic)
At the start: 15 parts, among them J1 Conn_01x02_Socket, J2 Conn_01x02_Socket, J3 J-jumper, P1 P-trim, U1 LM2596S-ADJ

Commit message: Second try routing.
Parts:
- J1: value Conn_01x02_Socket -> Vin
- J2: value Conn_01x02_Socket -> Vout
Other:
- moved on the sheet: C1, C2, D1, D2, J1, L1

Commit message: PCB design correction
Other:
- company: (none) -> Kroesch.NET
- title: (none) -> DC-Step-Down-Wandler für Raspberry Pi
Changed lines of the file:
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@@
 	(generator "eeschema")
 	(generator_version "9.0")
-	(paper "A4")
+	(paper "A5")
+	(title_block
+		(title "DC-Step-Down-Wandler für Raspberry Pi")
+		(date "2025-05-04")
+		(company "Kroesch.NET")
+	)
 	(junction
 		(at 104.14 95.25)
